File: lab1/lab1.sch (KiCad schematic (older format))
At the start: 15 parts

Commit message: lab 1
Parts:
- added C12, C16, C3: 100n, Capacitor_SMD:C_0805_2012Metric_Pad1.15x1.40mm_HandSolder, symbol Device:C
- added C13, C6: 10u, Capacitor_SMD:CP_Elec_4x5.4, symbol Device:CP
- added J1: USB_OTG, Connector_USB:USB_Mini-B_Wuerth_65100516121_Horizontal, symbol Connector:USB_OTG
- added J2: Conn_01x06_Male, Connector_PinHeader_2.54mm:PinHeader_1x06_P2.54mm_Horizontal, symbol Connector:Conn_01x06_Male
- added R3, R4: R, Resistor_SMD:R_0805_2012Metric_Pad1.15x1.40mm_HandSolder, symbol Device:R
- added U1: LM1117ADJ, Package_TO_SOT_SMD:SOT-223, symbol LM1117ADJ:LM1117ADJ
- C1, C10, C11, C14, C15, C2, C4, C5, C7, C8, C9: renamed from C?; footprint (none) -> Capacitor_SMD:C_0805_2012Metric_Pad1.15x1.40mm_HandSolder
- R1, R2: renamed from R?; footprint (none) -> Resistor_SMD:R_0805_2012Metric_Pad1.15x1.40mm_HandSolder
- Y1: renamed from Y?; footprint (none) -> Crystal:Crystal_HC49-U_Vertical
- gave numbers to parts that had none: 1
Connections:
- net +3V3: now also C12.1, C13.1, C16.1, J2.1 (Pin_1), R3.1, U1.2 (Vout1), U1.4 (Vout2)
- net GND: now also C12.2, C13.2, C16.2, C3.2, C6.2, J1.5 (GND), J1.6 (Shield), J2.3 (Pin_3), R4.2
- net SWDIO: now reaches U2.46 (PA13)
- net SWDIO: now also J2.4 (Pin_4)
- net SWCLK: now reaches U2.49 (PA14)
- net SWCLK: now also J2.2 (Pin_2)
- net SWO: now reaches U2.55 (PB3)
- net SWO: now also J2.6 (Pin_6)
- new net: R3.2, R4.1, U1.1 (ADJ)
- new net +5V: C3.1, C6.1, J1.1 (VBUS), U1.3 (Vin)
- no-connect marks 0 -> 50
