File: project/card/project/project.kicad_pcb (KiCad board)
At the start: 2 copper layers, 36 parts, among them J1 USB_OTG, J2 Conn_01x06_Male, J3 Conn_01x02_Male, J5 Conn_Coaxial, J6 Conn_01x07_Female, J7 Conn_01x05_Female, SW1 SW_Push, SW2 SW_Push, U1 LM1117ADJ, U2 CMWX1ZZABZ-078

Commit message: v1.0
Parts:
- removed RV1: R_POT, Potentiometer_THT:Potentiometer_Bourns_3386F_Vertical
- added Pot: R_POT, test:Potetio, F.Cu at (76.0, 83.0)
- moved R6 49.9 mm to (73.2, 82.1), turned to 180 degrees
- moved TV 11.9 mm to (49.0, 83.0)
- renumbered J5 to ANT, SW2 to Btn, J2 to Dbg, J7 to Dist, D2 to LED, D1 to LED, LS1 to Noise, SW1 to Rst, J6 to TV, J3 to UART, J1 to USB
Connections:
- U2 pad 24: /Pot -> /POT
Routing:
- net +3V3: track 151.8 -> 167.9 mm
- net /POT: track 0.00 -> 14.5 mm, vias 0 -> 1
- net /DataCom: track 37.1 -> 50.9 mm
- net Net-(J6-Pad3): track 24.4 -> 37.4 mm
- net Net-(J6-Pad4): track 18.8 -> 31.6 mm
- net /NSS: track 13.6 -> 26.4 mm
- net /Reset: track 29.8 -> 42.6 mm
- net Net-(R6-Pad1): track 0.00 -> 5.32 mm
- net /Pot: track 1.75 -> 0.00 mm
- net GND: track 15.4 -> 16.3 mm, vias 5 -> 7
- net /trig: track 16.1 -> 16.7 mm, vias 0 -> 2
